File: eagle_project/schematic.brd (EAGLE design)
At the start: 100 x 80 mm, 224 parts, among them IC2 AZ34063U, IC3 AZ34063U, IC4 LM358A, IC5 PIC24FJ64GU202-I_SS, IC6 LM358A, IC7 AZ34063U, J1 USB-B, Q1 16MHz, U1 OP07CD, U11 OP07CD, U12 OP07CD, U14 MCP4912-E/SL, U2 OP07CD, U3 OP07CD, U4 MCP1501T-40E/CHY, U5 OP07CD, U6 OP07CD, U7 OP07CD, U8 OP07CD, X4 MKDSN1,5/2-5,08, X5 MKDSN1,5/2-5,08, X6 MKDSN1,5/2-5,08, X7 MKDSN1,5/2-5,08, X8 MKDSN1,5/3-5,08

Commit message: changed R values in AO and changed DI
Parts:
- removed C41, C42, C9: 10n, rcl:C0805
- removed JP10, JP7: PINHD-2X4/90, Connector:2X04/90
- removed JP5, JP8: PINHD-1X5, Connector:1X05
- removed JP6, JP9: PINHD-2X6/90, Connector:2X06/90
- removed R61, R64: 10k, rcl:R0805
- removed R65: 2k4, rcl:R2010
- removed R70, R97: 1k, rcl:R0805
- added JP12, JP13: (no value), pinhead:2X04
- added JP14, JP15: (no value), pinhead:2X06
- added JP16, JP17: (no value), pinhead:1X05
- D1, D6, D7: value 1N4148 -> BZX55; device diode:MINIMELF -> diode:DO35Z10
- R21, R33: value 10k -> 750; device rcl:R0805 -> rcl:0309/12
- R31, R55: value 10k -> 600; device rcl:R0805 -> rcl:0309/12
- R32: value 2k4 -> 600; device rcl:R2010 -> rcl:0309/12
- R56: value 2k4 -> 750; device rcl:R2010 -> rcl:0309/12
- R67, R77, R78, R79, R81, R82, R84, R87: value 1k -> 100k
- R80, R95: value 220 -> 22k
- R83, R85, R89, R90: value 1.44k -> 144k
- R86, R88: value 3.88k -> 388k
- moved D6 282.1 mm to (-121.9, -109.2)
- moved R55 275.0 mm to (-104.1, -108.0)
- moved D1 270.5 mm to (-121.9, -96.5)
- moved R33 266.7 mm to (-104.1, -101.6)
- moved D7 262.3 mm to (-121.9, -90.2)
- moved R56 257.9 mm to (-104.1, -114.3)
- moved R31 254.1 mm to (-104.1, -88.9)
- moved R21 250.4 mm to (-104.1, -82.5)
- moved R32 219.9 mm to (-104.1, -95.2)
- moved C25 155.6 mm to (-127.0, -21.6)
- moved R73 155.6 mm to (-123.2, -16.5)
- moved R77 155.6 mm to (-95.2, -21.6)
- moved R79 155.6 mm to (-127.0, -27.9)
- moved R90 155.6 mm to (-101.6, -21.6)
- moved R98 155.6 mm to (-95.2, -27.9)
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Connections:
- new net N$115: OK4.1, R21.2
- net +5V: no longer C41.1, C42.1, C9.1, OK1.1, OK2.1, OK4.1, R21.2, R31.2, R33.2, R55.2, R61.2, R64.2, X5.1, X6.1, X7.1
- net D_IN_0: no longer R31.1
- net D_IN_1: no longer R55.1
- net D_IN_2: no longer R64.1
- net GND: now also JP12.7, JP12.8, JP13.7, JP13.8, JP14.11, JP14.12, JP15.11, JP15.12; no longer JP10.7, JP10.8, JP6.11, JP6.12, JP7.7, JP7.8, JP9.11, JP9.12
- net I+: now also JP16.1, JP17.1; no longer JP5.1, JP8.1
- net I-: now also JP16.2, JP17.2; no longer JP5.2, JP8.2
- net N$100: now also JP15.8; no longer JP9.8
- net N$101: now also JP15.10; no longer JP9.10
- net N$105: now also JP14.8; no longer JP6.8
- net N$106: now also JP14.10; no longer JP6.10
- net N$13: now also R32.1, X6.1; no longer C9.2, D1.A, OK4.2, R21.1
- net N$17: now also D1.A, OK1.2, X6.2; no longer R32.1, X5.2
- net N$21: now also R33.1
- net N$29: now also OK1.1, R33.2; no longer C41.2, D6.A, OK1.2, R33.1
- net N$36: now also R31.1, X5.1; no longer R56.1, X6.2
- net N$39: now also D6.A, OK4.2, X5.2; no longer D6.C, R56.2
- net N$54: now also R55.1, X7.1; no longer C42.2, D7.A, OK2.2, R61.1
- net N$57: now also D7.A, OK2.2; no longer R65.1
- net N$61: now also R55.2, R56.1; no longer R65.2
- net N$67: now also OK2.1, R56.2; no longer R97.1, T4.B
- net N$68: now also JP13.4; no longer JP7.4
- net N$71: now also JP14.3; no longer JP6.3
- net N$72: now also JP14.7; no longer JP6.7
- net N$73: now also JP14.9; no longer JP6.9
- net N$74: now also JP14.5; no longer JP6.5
- net N$75: now also JP13.1; no longer JP7.1
- net N$76: now also JP13.3, JP14.1; no longer JP6.1, JP7.3
- net N$77: now also JP13.5, JP14.2; no longer JP6.2, JP7.5
- net N$78: now also JP13.6, T4.B; no longer JP7.6, R97.2
- net N$80: now also JP14.6; no longer JP6.6
- net N$81: now also JP14.4; no longer JP6.4
- net N$84: now also D6.C, R21.1, R31.2; no longer R70.1, T3.B
- net N$85: now also JP12.4; no longer JP10.4
- net N$86: now also JP15.3; no longer JP9.3
- net N$87: now also JP15.7; no longer JP9.7
- net N$88: now also JP15.9; no longer JP9.9
- net N$90: now also JP15.5; no longer JP9.5
- net N$91: now also JP12.1; no longer JP10.1
- net N$92: now also JP12.3, JP15.1; no longer JP10.3, JP9.1
- net N$94: now also JP12.5, JP15.2; no longer JP10.5, JP9.2
- net N$95: now also JP12.6, T3.B; no longer JP10.6, R70.2
- net N$98: now also JP15.6; no longer JP9.6
- net N$99: now also JP15.4; no longer JP9.4
- net V+: now also JP12.2, JP13.2, JP16.3, JP17.3; no longer JP10.2, JP5.3, JP7.2, JP8.3
- net V-: now also JP16.4, JP16.5, JP17.4, JP17.5; no longer JP5.4, JP5.5, JP8.4, JP8.5

Commit message: Reverted DI. Added linear +-12V PSU with transformer
Parts:
- removed C11: 1n, rcl:C0805
- removed C12: 100uF/25V/105°, rcl:E2-5
- removed D2: SS13+, diode:SMC
- removed IC2: AZ34063U, IMPORTED_ELEMENTS:SO08
- removed L6: 1uH, IMPORTED:R0805
- removed L7: 1mH, SamacSys_Parts:12LRS105C
- removed LED10, LED9: (no value), led:CHIPLED_0805
- removed LED3: (no value), led:LED3MM
- removed R104, R105: 1k, rcl:R0805
- removed R33, R56: 750, rcl:0309/12
- removed R35: (no value), rcl:R0805
- removed R36: 953R, rcl:R0805
- removed R37: 8k2, rcl:R0805
- removed R38: 0R39, rcl:R0805
- removed R55: 600, rcl:0309/12
- removed S3: (no value), switch:TL3XPO
- added C41, C42, C9: 100n, rcl:C0805
- added C43, C44, C45: 0.1u, rcl:C0805
- added D10: 1N4001-T, SamacSys_Parts:DIOAD1408W86L464D236
- added D8: 1N4148, diode:MINIMELF
- added IC1: L7912CV-DG, SamacSys_Parts:TO255P460X1020X2008-3P
- added Q2: L7812ABV-DG, SamacSys_Parts:TO255P460X1020X2008-3P
- added TR1: TRANSFORMER-PCB-2X12, DelavnicaCustomComponents:TRANSFORMER-PCB-2X12_FOOTPRINT
- added U$1: 2828XX-2282837-2, Connector:TERMBLK_508-2N
- added U9: DF01S, SamacSys_Parts:SOT508P985X260-4N
- C10: value 1000uF/25V/105° -> 6000uF; device rcl:E5-13 -> rcl:EB22,5D
- C2: value 100nF -> 6000uF; device rcl:C0805 -> rcl:EB22,5D
- D1, D6: value BZX55 -> 1N4148; device diode:DO35Z10 -> diode:MINIMELF
- D7: value BZX55 -> 1N4001-T; device diode:DO35Z10 -> SamacSys_Parts:DIOAD1408W86L464D236
- R21: value 750 -> 1k; device rcl:0309/12 -> rcl:R2512
- R31, R32: value 600 -> 1k; device rcl:0309/12 -> rcl:R2512
- moved C2 452.2 mm to (-222.2, -285.8)
- moved C10 392.9 mm to (-222.2, -308.6)
- moved D7 211.3 mm to (-229.9, -271.8)
- moved R21 150.9 mm to (-2.80, -194.3)
- moved R32 150.9 mm to (-2.80, -207.0)
- moved R31 137.3 mm to (-2.80, -181.6)
- moved D6 66.1 mm to (-162.6, -161.3)
- moved D1 61.2 mm to (-162.6, -142.2)
Connections:
- removed net +5V2: C10.-, C11.2, D2.A, IC2.4, L6.1, R36.2
- removed net N$120: LED10.A, R105.1
- removed net N$19: LED3.K, R35.1
- removed net N$31: IC2.5, R36.1, R37.2
- removed net N$33: IC2.1, IC2.7, IC2.8, R38.2
- removed net N$34: C11.1, IC2.3
- removed net N$42: D2.C, IC2.2, L7.1
- removed net PROG: R105.2, S3.1
- removed net RUN: R104.2, S3.3
- new net N$121: C43.1, TR1.S11, U9.4
- new net N$122: C43.2, TR1.S22, U9.3
- new net N$123: D8.C, X5.2
- new net N$124: C2.+, Q2.1, U9.1
- new net N$125: C10.-, IC1.2, U9.2
- net +12V: now also C44.1, D10.1, Q2.3; no longer C2.1, IC2.6, R38.1
- net -12V: now also C45.2, D7.2, IC1.3; no longer C12.-, L6.2, R35.2
- net GND: now also C2.-, C44.2, C45.1, D10.2, D7.1, IC1.1, Q2.2, TR1.S12, TR1.S21; no longer C12.+, C2.2, L7.3, LED10.C, LED3.A, LED9.C, R37.1
- net N$115: now also TR1.P2, U$1.1; no longer OK4.1, R21.2
- net N$119: now also TR1.P1, U$1.2; no longer LED9.A, R104.1
- net N$13: now also R21.1; no longer R32.1
- net N$17: now also C41.1, OK1.1, R21.2; no longer D1.A, OK1.2, X6.2
- net N$21: now also C41.2, D1.A, OK1.2; no longer D1.C, R32.2, R33.1
- net N$29: now also D1.C, X6.2; no longer OK1.1, R33.2
- net N$39: now also C9.2, D8.A; no longer D6.A, X5.2
- net N$54: now also R32.1; no longer R55.1
- net N$57: now also C42.1, OK2.1, R32.2; no longer D7.A, OK2.2, X7.2
- net N$61: now also C42.2, D6.A, OK2.2; no longer D7.C, R55.2, R56.1
- net N$67: now also D6.C, X7.2; no longer OK2.1, R56.2
- net N$84: now also C9.1, OK4.1; no longer D6.C, R21.1
- net VCC: no longer S3.2
